Commit message: sistemazioni

File: urdf/ur10_sim.urdf.xacro (robot description, xacro)
@@ -44,3 +44,52 @@
     <origin xyz="0.0 0.0 0.0" rpy="0.0 0.0 0.0" />
   </joint>
+    <!-- Spawn user camera -->
+    <link name="camera_link"/>
+    <!-- Attach camera to tool0 -->
+    <joint name="camera" type="fixed">
+      <origin xyz="0 -0.000447 0.08739618542" rpy="0 ${-pi/2} ${pi/2}" />
+      <parent link="tool0" />
+      <child link="camera_link" />
+    </joint>
+<gazebo reference="camera_link">
+  <sensor name="rgbd" type="depth">
+    <update_rate>100</update_rate>
+    <camera>
+      <horizontal_fov>1.047198</horizontal_fov>
+      <image>
+        <width>1080</width>
+        <height>680</height>
+        <format>R8G8B8</format>
+      </image>
+      <clip>
+        <near>0.005</near>
+        <far>10</far>
+      </clip>
+    </camera>
+    <plugin name="camera_controller" filename="libgazebo_ros_openni_kinect.so">
+      <baseline>0.2</baseline>
+      <alwaysOn>true</alwaysOn>
+      <updateRate>1.0</updateRate>
+      <cameraName>camera_ir</cameraName>
+      <imageTopicName>/camera/color/image_raw</imageTopicName>
+      <cameraInfoTopicName>/camera/color/camera_info</cameraInfoTopicName>
+      <depthImageTopicName>/camera/depth/image_raw</depthImageTopicName>
+      <depthImageInfoTopicName>/camera/depth/camera_info</depthImageInfoTopicName>
+      <pointCloudTopicName>/camera/depth/points</pointCloudTopicName>
+      <frameName>cameradepth_link</frameName>
+      <pointCloudCutoff>0.5</pointCloudCutoff>
+      <pointCloudCutoffMax>3.0</pointCloudCutoffMax>
+      <distortionK1>0.00000001</distortionK1>
+      <distortionK2>0.00000001</distortionK2>
+      <distortionK3>0.00000001</distortionK3>
+      <distortionT1>0.00000001</distortionT1>
+      <distortionT2>0.00000001</distortionT2>
+      <CxPrime>0</CxPrime>
+      <Cx>0</Cx>
+      <Cy>0</Cy>
+      <focalLength>0</focalLength>
+      <hackBaseline>0</hackBaseline>
+    </plugin>
+  </sensor>
+</gazebo>
 </robot>

Commit message: ravenna

File: urdf/ur10_sim.urdf.xacro (robot description, xacro)
@@ -48,5 +48,5 @@
     <!-- Attach camera to tool0 -->
     <joint name="camera" type="fixed">
-      <origin xyz="0 -0.000447 0.08739618542" rpy="0 ${-pi/2} ${pi/2}" />
+      <origin xyz="0 0 0" rpy="0 ${-pi/2} ${pi/2}" />
       <parent link="tool0" />
       <child link="camera_link" />
@@ -55,5 +55,5 @@
     <!-- Attach camera to tool0 -->
     <joint name="camera_depth" type="fixed">
-      <origin xyz="0 0 0" rpy="${pi/2} ${0} ${pi/2}" />
+      <origin xyz="0 0 0" rpy="${-pi/2} ${0} ${-pi/2}" />
       <parent link="camera_link" />
       <child link="cameradepth_link" />

File: urdf/ur5_sim.urdf.xacro (robot description, xacro)
@@ -20,5 +20,5 @@
     <color rgba="1 1 1 1"/>
   </material>
-  <link name="table">
+  <!--link name="table">
     <visual>
       <geometry>
@@ -37,5 +37,5 @@
     <child link="table"/>
     <origin xyz="0.0 0.0 -0.01" rpy="0 0 0"/>
-  </joint>
+  </joint-->
   <link name="world" />
   <joint name="world_joint" type="fixed">
