Commit message: dopo un po

File: urdf/ur10_ufficiale.xacro (robot description, xacro)
@@ -49,5 +49,5 @@
     <joint name="camera" type="fixed">
       <!--origin xyz="0 0 0" rpy="0 ${-pi/2} ${pi/2}" /-->
-      <origin xyz="0.35 0.1 0.37" rpy="${0} ${0} ${5*pi/8}" />
+      <origin xyz="-0.4 0 -0.1" rpy="${-pi/2} ${-pi/8} ${0}" />
       <!--parent link="tool0" /-->
       <parent link="base_link" />
